File: General Data/Park PCB/PARKPCB.sch (EAGLE design)
At the start: 3 parts, among them M1 ETHERNET-ENC28J60

Commit message: Trabajando en el PCB
Parts:
- removed U$1: ARDUINO-TEENSY++, teensypp:ARDUINO-TEENSY++
- added 3.3V, 3.3V1, 5V: LSP10, solpad:LSP10
- added C5V, C5V1, CUCAP, CXTAL1, CXTAL2, CXTAL3, CXTAL4: 1u, rcl:C-US050-030X075
- added CAREF, CAREF1, CAREF2, CAREF3: 0.1U, rcl:C-US050-030X075
- added IC1: (no value), controller-micro_atmel_jd:AT90USB-TQFP
- added JP1: (no value), adafruit:PINHD-1X3
- added Q1: 16M, special:XTAL/S
- added Q2: 32768, special:XTAL/S
- added RALE: 1k, rcl:R-US_0309/12
- added RD+, RD-, RD-1: 22, rcl:R-US_0309/12
- added RESET: (no value), adafruit:SWITCH_PUSHBUTTONC&K_KSS
- added U1: MCP1825_SOT223, bt_regulator:MCP1825_SOT223
- added X1: USB-MB-S, con-usb:USB-MB-S
Connections:
- removed net E0: U$1.8
- removed net E1: U$1.9
- removed net RX: U$1.2,RX,INT2
- removed net SCLK: U$1.21
- removed net T1: U$1.10
- removed net T2: U$1.11
- removed net T3: U$1.12
- removed net T4: U$1.13
- removed net T5: U$1.14,PWM
- removed net T6: U$1.15,PWM
- removed net T7: U$1.16,PWM
- removed net T8: U$1.17
- removed net TX: U$1.3,TX,INT3
- new net +3V3: 3.3V.MP, 3.3V1.MP, C5V1.1, CAREF1.1, CAREF2.1, CAREF3.1, CUCAP.1, IC1.AVCC, IC1.UCAP, IC1.VCC, IC1.VCC@1, JP1.1, U1.VOUT
- new net A0: IC1.PA0_AD0
- new net A1: IC1.PA1_AD1
- new net A2: IC1.PA2_AD2
- new net A3: IC1.PA3_AD3
- new net A4: IC1.PA4_AD4
- new net A5: IC1.PA5_AD5
- new net A6: IC1.PA6_AD6
- new net A7: IC1.PA7_AD7
- new net ALE: RALE.2
- new net C0: IC1.PC0_A8
- new net C1: IC1.PC1_A9
- new net C2: IC1.PC2_A10
- new net C3: IC1.PC3_A11_T3
- new net C4: IC1.PC4_A12_OC3C
- new net C5: IC1.PC5_A13_OC3B
- new net C6: IC1.PC6_A14_OC3A
- new net C7: IC1.PC7_A15_IC3_CLK0
- new net E4: CXTAL4.1, IC1.PE4_INT4_TOSC1, Q2.2
- new net E5: CXTAL3.1, IC1.PE5_INT5_TOSC2, Q2.1
- new net INTE: M1.INT
- new net N$11: IC1.D+, RD+.2
- new net N$13: CXTAL2.1, IC1.XTAL2, Q1.1
- new net N$14: CXTAL1.1, IC1.XTAL1, Q1.2
- new net N$15: IC1.PF0_ADC0, JP1.2, RD-1.1
- new net N$7: IC1.D-, RD-.2
- new net N$8: RD+.1, X1.D+
- new net RESET: IC1./RESET, RESET.P$1
- new net TRIGGERBC: IC1.PF1_ADC1
- new net TXBC: IC1.PD2_RXD1_INT2
- net GND: now also C5V.2, C5V1.2, CAREF.2, CAREF1.2, CAREF2.2, CAREF3.2, CUCAP.2, CXTAL1.2, CXTAL2.2, CXTAL3.2, CXTAL4.2, IC1.AGND, IC1.GND, IC1.GND@1, IC1.UGND, JP1.3, RALE.1, RD-1.2, RESET.P$2, U1.GND, X1.GND; no longer U$1.GND
- net MISO: now also M1.SO; no longer U$1.23
- net MOSI: now also M1.SI; no longer U$1.22
- net N$2: now also CAREF.1, IC1.AREF; no longer M1.CS
- net N$4: now also 5V.MP, C5V.1, IC1.UVCC, IC1.VBUS, U1.VIN, X1.VBUS; no longer M1.SI
- net N$6: now also RD-.1, X1.D-; no longer M1.SO
- net SCL: no longer U$1.0,PWM,INT0
- net SDA: no longer U$1.1,PWM,INT1
- net SS: now also M1.CS; no longer U$1.20
