File: General Data/projects/Park PCB/ESPswitch.brd (EAGLE design)
At the start: 160 x 100 mm, 9 parts, among them T1 2N2222, T2 2N2222

Commit message: Actualización de PCBs
Parts:
- added GND, VCC: (no value), adafruit:1X01
- moved D1 3.00 mm to (23.4, 17.9)
- moved ESP8266 3.00 mm to (11.0, 14.2)
- moved R1 3.00 mm to (10.7, 19.9)
- moved R2 3.00 mm to (11.0, 11.7)
- moved R3 3.00 mm to (10.7, 23.8)
- moved RELE 3.00 mm to (20.9, 26.9)
- moved T1 3.00 mm to (9.43, 28.8)
- moved VREG 3.00 mm to (9.21, 41.5)
- moved T2 3.00 mm to (9.43, 17.4)
Connections:
- net GND: now also GND.1
- net VCC: now also VCC.1
Routing:
- net GND: track 33.5 -> 38.8 mm
- net VCC: track 17.5 -> 21.3 mm
- net +3V3: track 48.5 -> 47.9 mm
