File: General Data/projects/Park PCB/PARKPCB.brd (EAGLE design)
At the start: 160 x 100 mm, 58 parts, among them J1 MAGJACK, Q1 16M, Q2 16M, X1 22-23-2041

Commit message: Actualización de PCBs
Parts:
- removed BARCODESCANNER, PRINTER1, PRINTER2: RJ45, RJ45 Jack:RJ45
- added BARCODE, SSERIAL1, SSERIAL2: RJ45-6L-B, con-tycoelectronics:RJ45-NO-SHIELD
- PRINTER: value RJ45 -> RJ45-6L-B; device RJ45 Jack:RJ45 -> con-tycoelectronics:RJ45-NO-SHIELD
- moved PRINTER 10.3 mm to (8.00, 27.0), turned to 270 degrees
Connections:
- net +3V3: now also BARCODE.4; no longer BARCODESCANNER.P$10
- net GND: now also BARCODE.1, PRINTER.1; no longer BARCODESCANNER.P$8, PRINTER.P$8
- net SRX1: now also SSERIAL1.1; no longer PRINTER1.P$8
- net SRX2: now also SSERIAL2.1; no longer PRINTER2.P$8
- net STX1: now also SSERIAL1.2; no longer PRINTER1.P$3
- net STX2: now also SSERIAL2.2; no longer PRINTER2.P$3
- net T1OUT: now also PRINTER.2; no longer PRINTER.P$3
- net TRIGGERBC: now also BARCODE.3; no longer BARCODESCANNER.P$9
- net TXBC: now also BARCODE.2; no longer BARCODESCANNER.P$3
Routing:
- net GND: track 142.1 -> 203.4 mm, vias 16 -> 17
- net STX2: track 88.4 -> 74.1 mm
- net SRX2: track 92.4 -> 79.5 mm
- net +3V3: track 288.3 -> 285.8 mm
- net TXBC: track 133.1 -> 134.5 mm
- net SCLK: track 28.7 -> 30.1 mm
- net TRIGGERBC: track 98.2 -> 99.5 mm
- net STX1: track 98.7 -> 99.5 mm
- net SRX1: track 109.6 -> 110.4 mm
- net XTAL2: track 6.93 -> 7.51 mm
- net D+IN: vias 2 -> 1
- added copper zone on layer 16, net GND
- removed copper zone on layer 1, net GND
