File: General Data/projects/Park PCB/PARKPCB.sch (EAGLE design)
At the start: 58 parts, among them J1 MAGJACK, Q1 16M, Q2 16M, X1 22-23-2041

Commit message: Actualización de PCBs
Parts:
- removed BARCODESCANNER, PRINTER1, PRINTER2: RJ45, RJ45 Jack:RJ45
- added BARCODE, SSERIAL1, SSERIAL2: RJ45-6L-B, con-tycoelectronics:RJ45-6L-B
- PRINTER: value RJ45 -> RJ45-6L-B; device RJ45 Jack:RJ45 -> con-tycoelectronics:RJ45-6L-B
Connections:
- net +3V3: now also BARCODE.4; no longer BARCODESCANNER.PIN4
- net GND: now also BARCODE.1, PRINTER.1; no longer BARCODESCANNER.PIN1, PRINTER.PIN1
- net SRX1: now also SSERIAL1.1; no longer PRINTER1.PIN1
- net SRX2: now also SSERIAL2.1; no longer PRINTER2.PIN1
- net STX1: now also SSERIAL1.2; no longer PRINTER1.PIN2
- net STX2: now also SSERIAL2.2; no longer PRINTER2.PIN2
- net T1OUT: now also PRINTER.2; no longer PRINTER.PIN2
- net TRIGGERBC: now also BARCODE.3; no longer BARCODESCANNER.PIN3
- net TXBC: now also BARCODE.2; no longer BARCODESCANNER.PIN2
