File: General Data/projects/Park PCB/PARKPCBTEENSY.sch (EAGLE design)
At the start: 56 parts, among them J1 MAGJACK, Q1 16M, Q2 16M, X1 22-23-2041

Commit message: Actualización de PCBs
Parts:
- removed +3V3P, +5VP, GND: LSP10, solpad:LSP10
- removed AT90USB1286: AT90USB1286-AU, Atmel_By_element14_Batch_1-00:AT90USB1286-AU
- removed BARCODESCANNER, PRINTER, PRINTER1, PRINTER2: RJ45, RJ45 Jack:RJ45
- removed BOTON: 22-23-2021, con-molex:22-23-2021
- removed C10, CETH: 100n, rcl:C-US050-030X075
- removed C5V, CUCAP, CXTAL1, CXTAL2: 1u, rcl:C-US050-030X075
- removed C8, CAREF1, CAREF2, CAREF3: 0.1u, rcl:C-US050-030X075
- removed C9: 10u, rcl:CPOL-USB45181B
- removed CAREF: 0.1U, rcl:C-US050-030X075
- removed CETH1: 10n, rcl:C-US050-030X075
- removed COSC1, COSC2: 18p, rcl:C-US050-030X075
- removed ETHERNECHIP: ENC28J60-I/SP, microchip-ethernet:ENC28J60-I/SP
- removed FB/0805/600: FERRITE_0805, audio amplifier example:FERRITE_0805
- removed ICL3232: ICL3232, ICL3232:ICL3232
- removed J1: MAGJACK, SparkFun-Connectors:MAGJACK
- removed Q1, Q2: 16M, special:XTAL/S
- removed RALE: 1k, rcl:R-US_0309/12
- removed RBIAS: 2.2k, rcl:R-US_0309/12
- removed RCS: 100k, rcl:R-US_0309/12
- removed RD+, RD-: 22, rcl:R-US_0309/12
- removed RESET: (no value), adafruit:SWITCH_PUSHBUTTONC&K_KSS
- removed RETH1, RETH2, RETH3, RETH4: 49.9, rcl:R-US_0309/12
- removed RLEDA, RLEDB: 180, rcl:R-US_0309/12
- removed RRST: 10k, rcl:R-US_0309/12
- removed USB: USB-MB-S, con-usb:USB-MB-S
- removed VREG: LM1086TO263, v-reg-2:LM1086TO263
- removed X1: 22-23-2041, con-molex:22-23-2041
- added BARCODE, LCD: (no value), con-lstb:MA04-1
- added BUTTON: 22-23-2021, con-molex:22-23-2021
- added KEYBOARD: (no value), adafruit:PINHD-1X8BIG
- added M1: ETHERNET-ENC28J60, diy-modules:ETHERNET-ENC28J60
- added SERIAL1, SERIAL2, SERIAL3: RJ45-6L-B, con-tycoelectronics:RJ45-6L-B
- added U$1: ARDUINO-TEENSY++, teensypp:ARDUINO-TEENSY++
- added U$2: LM1086TO220V, v-reg-2:LM1086TO220V
- added U$3: ICL3232, ICL3232:ICL3232
- C1, C2: value 0.1u -> 100u; device rcl:C-US050-030X075 -> rcl:CPOL-USB45181B
- C3, C4, C5, C6, C7: value 0.1u -> 1u; device rcl:C-US050-030X075 -> rcl:CPOL-USB45181B
- JP1: device adafruit:PINHD-1X8BIG -> adafruit:PINHD-1X1
Connections:
- removed net ALE: AT90USB1286.PE2, RALE.2
- removed net AREF: AT90USB1286.AREF, CAREF.1
- removed net BOTON1: AT90USB1286.PE0, BOTON-1.S
- removed net BOTON2: AT90USB1286.PE1, BOTON-2.S
- removed net D+: AT90USB1286.D+, RD+.2
- removed net D+IN: RD+.1, USB.D+
- removed net D-: AT90USB1286.D-, RD-.2
- removed net D-IN: RD-.1, USB.D-
- removed net LEDA: ETHERNECHIP.LEDA, J1.YLED+
- removed net LEDB: ETHERNECHIP.LEDB, J1.GLED+
- removed net N$20: C1.1, ICL3232.C1+
- removed net N$21: C3.1, ICL3232.V+
- removed net N$22: C1.2, ICL3232.C1-
- removed net N$23: C2.1, ICL3232.C2+
- removed net N$24: C2.2, ICL3232.C2-
- removed net N$25: C4.2, ICL3232.V-
- removed net OSC1: COSC1.1, ETHERNECHIP.OSC1, Q2.1
- removed net OSC2: COSC2.1, ETHERNECHIP.OSC2, Q2.2
- removed net RESET: AT90USB1286.~RESET, RESET.P$1
- removed net RST: ETHERNECHIP.RESET, RRST.1
- removed net SCLK: AT90USB1286.PB1, ETHERNECHIP.SCK
- removed net SRX1: AT90USB1286.PB4, PRINTER1.PIN1
- removed net SRX2: AT90USB1286.PB6, PRINTER2.PIN1
- removed net STX1: AT90USB1286.PB5, PRINTER1.PIN2
- removed net STX2: AT90USB1286.PB7, PRINTER2.PIN2
- removed net T0: AT90USB1286.PC0, JP1.1
- removed net T1: AT90USB1286.PC1, JP1.2
- removed net T1IN: AT90USB1286.PD3, ICL3232.T1IN
- removed net T2: AT90USB1286.PC2, JP1.3
- removed net T3: AT90USB1286.PC3, JP1.4
- removed net T4: AT90USB1286.PC4, JP1.5
- removed net T5: AT90USB1286.PC5, JP1.6
- removed net T6: AT90USB1286.PC6, JP1.7
- removed net T7: AT90USB1286.PC7, JP1.8
- removed net TPIN+: ETHERNECHIP.TPIN+, J1.RD+, RETH3.1
- removed net TPIN-: ETHERNECHIP.TPIN-, J1.RD-, RETH4.1
- removed net TPOUT+: ETHERNECHIP.TPOUT+, J1.TD+, RETH2.1
- removed net TPOUT-: ETHERNECHIP.TPOUT-, J1.TD-, RETH1.1
- removed net TXBC: AT90USB1286.PD2, BARCODESCANNER.PIN2
- removed net XTAL1: AT90USB1286.XTAL1, CXTAL1.1, Q1.2
- removed net XTAL2: AT90USB1286.XTAL2, CXTAL2.1, Q1.1
- new net BARRERA: JP1.1, U$1.40,A2
- new net N$10: KEYBOARD.8, U$1.10
- new net N$11: C3.+, U$3.C1+
- new net N$12: C4.+, U$3.V+
- new net N$13: C3.-, U$3.C1-
- new net N$16: C5.-, U$3.V-
- new net N$8: KEYBOARD.6, U$1.12
- new net N$9: KEYBOARD.7, U$1.11
- new net RX: BARCODE.4, U$1.2,RX,INT2
- new net RXS1: SERIAL1.1, U$1.24,PWM
- new net RXS2: SERIAL2.1, U$1.26,PWM
- new net SCK: M1.SCK, U$1.21
- new net TX: U$1.3,TX,INT3, U$3.T1IN
- new net TXS1: SERIAL1.2, U$1.25,PWM
- new net TXS2: SERIAL2.2, U$1.27,PWM
- net +3V3: now also BARCODE.1, C1.+, C7.+, M1.3V3, M1.RST, U$1.VCC, U$2.OUT, U$3.VCC; no longer +3V3P.MP, AT90USB1286.AVCC, AT90USB1286.UCAP, AT90USB1286.VCC, AT90USB1286.VCC_2, BARCODESCANNER.PIN4, C10.1, C5.1, CAREF1.1, CAREF2.1, CAREF3.1, CUCAP.1, ETHERNECHIP.VDD, ETHERNECHIP.VDDOSC, FB/0805/600.P$1, ICL3232.VCC, RCS.2, RRST.2, VREG.OUT
- net +5V: now also C2.+, LCD.2, U$1.+5V, U$2.IN; no longer +5VP.MP, AT90USB1286.UVCC, AT90USB1286.VBUS, C5V.1, USB.VBUS, VREG.IN, X1-4.S
- net GND: now also BARCODE.2, C1.-, C2.-, C4.-, C5.+, C7.-, LCD.1, M1.GND.1, SENSORPAPEL.2, SERIAL3.2, U$1.GND, U$2.GND, U$3.GND; no longer AT90USB1286.GND, AT90USB1286.GND_2, AT90USB1286.GND_3, AT90USB1286.UGND, BARCODESCANNER.PIN1, C10.2, C3.2, C4.1, C5.2, C5V.2, C6.2, C7.2, C8.2, C9.-, CAREF.2, CAREF1.2, CAREF2.2, CAREF3.2, CETH.2, CETH1.2, COSC1.2, COSC2.2, CUCAP.2, CXTAL1.2, CXTAL2.2, ETHERNECHIP.VSS, ETHERNECHIP.VSSOSC, ETHERNECHIP.VSSPLL, ETHERNECHIP.VSSRX, ETHERNECHIP.VSSTX, GND.MP, ICL3232.GND, PRINTER.PIN1, RALE.1, RBIAS.2, RESET.P$2, RLEDA.2, RLEDB.2, SENSORPAPEL.3, USB.GND, VREG.GND, X1-1.S
- net INTE: now also M1.INT, U$1.19; no longer AT90USB1286.PE7, ETHERNECHIP.INT
- net MISO: now also M1.SO, U$1.23; no longer AT90USB1286.PB3, ETHERNECHIP.SO
- net MOSI: now also M1.SI, U$1.22; no longer AT90USB1286.PB2, ETHERNECHIP.SI
- net N$1: now also BUTTON-1.S, U$1.9; no longer CETH.1, FB/0805/600.P$2, J1.TCT, RETH1.2, RETH2.2
- net N$14: now also C6.+, U$3.C2+; no longer J1.GLED-, RLEDB.1
- net N$15: now also C6.-, U$3.C2-; no longer J1.YLED-, RLEDA.1
- net N$2: now also BUTTON-2.S, U$1.8; no longer C6.1, ETHERNECHIP.VDDPLL
- net N$3: now also KEYBOARD.1, U$1.17; no longer C7.1, ETHERNECHIP.VDDTX
- net N$4: now also KEYBOARD.2, U$1.16,PWM; no longer C8.1, ETHERNECHIP.VDDRX
- net N$5: now also KEYBOARD.3, U$1.15,PWM; no longer CETH1.1, RETH3.2, RETH4.2
- net N$6: now also KEYBOARD.4, U$1.14,PWM; no longer C9.+, ETHERNECHIP.VCAP
- net N$7: now also KEYBOARD.5, U$1.13; no longer ETHERNECHIP.RBIAS, RBIAS.1
- net PAPEL: now also SENSORPAPEL.3, U$1.38,A0; no longer AT90USB1286.PF0, SENSORPAPEL.2
- net SCL: now also LCD.4, U$1.0,PWM,INT0; no longer AT90USB1286.PD0, X1-2.S
- net SDA: now also LCD.3, U$1.1,PWM,INT1; no longer AT90USB1286.PD1, X1-3.S
- net SS: now also M1.CS, U$1.20; no longer AT90USB1286.PB0, ETHERNECHIP.CS, RCS.1
- net T1OUT: now also SERIAL3.1, U$3.T1OUT; no longer ICL3232.T1OUT, PRINTER.PIN2
- net TRIGGERBC: now also BARCODE.3, U$1.39,A1; no longer AT90USB1286.PF1, BARCODESCANNER.PIN3
Other:
- moved on the sheet: RPAPEL, SENSORPAPEL
