File: General Data/projects/ParticlePCB/ParticlePCB.sch (EAGLE design)
At the start: 11 parts, among them X1 RJ45-6L-B

Commit message: Actualización de PCBs
Parts:
- removed AUDIT: 53047-05, PNP:53047-05
- removed RSCL2: 10k, rcl:R-US_0207/10
- added MEMAUDIT: 53047-06, PNP:53047-06
Connections:
- removed net BLK: AUDIT-4.S, U$2.WKP
- removed net N$2: AUDIT-5.S, RSCL2.1
- removed net N$3: U$2.DAC, X1.3
- removed net N$4: U$2.A5, X1.4
- removed net N$5: U$2.A4, X1.5
- removed net N$6: U$2.A3, X1.6
- removed net N$7: U$2.A2, X1.7
- new net MISO: MEMAUDIT-3.S, U$2.A4
- new net MOSI: MEMAUDIT-2.S, U$2.A5
- new net SCK: MEMAUDIT-4.S, U$2.A3
- new net SS: MEMAUDIT-5.S, U$2.A2
- net +3V3: now also MEMAUDIT-6.S; no longer RSCL2.2
- net GND: now also MEMAUDIT-1.S; no longer AUDIT-1.S
- net RX: now also X1.4; no longer AUDIT-3.S
- net TX: now also X1.3; no longer AUDIT-2.S
Other:
- moved on the sheet: X1

Commit message: Actualiazndo PCBs
Parts:
- removed G1: CH23-1220LF, battery:CH23-1220LF
- removed RSCL1: 10k, rcl:R-US_0207/10
- added BT1: 3V, SparkFun-Batteries:BATTERY-12MM_PTH
- added JP1, JP11, JP12, JP13, JP2, JP3, JP4, JP6, JP7, JP8: (no value), adafruit:PINHD-1X1CB
Connections:
- removed net N$1: PRINTER-1.S, RSCL1.2
- new net D4: U$2.D4, X1.8
- net +3V3: now also X1.2, X1.3
- net +5V: now also PRINTER-5.S; no longer RSCL1.1
- net DTR: now also PRINTER-2.S, U$2.WKP; no longer PRINTER-3.S, U$2.D4
- net GND: now also BT1.-, JP11.1, JP12.1, JP3.1, JP4.1, JP7.1, JP8.1, PRINTER-1.S, X1.7; no longer G1.-, PRINTER-5.S, X1.2
- net RX: now also PRINTER-3.S; no longer X1.4
- net RXP: now also X1.4; no longer PRINTER-2.S
- net TX: now also PRINTER-4.S; no longer X1.3
- net TXP: now also X1.6; no longer PRINTER-4.S
- net VBAT: now also BT1.+, JP1.1, JP13.1, JP2.1, JP6.1; no longer G1.+
Other:
- moved on the sheet: PRINTER-2, PRINTER-3
